File: sd_tos_hw/sd_tos_dip28.brd (EAGLE design)
At the start: 19.5 x 63.5 mm, 20 parts, among them IC1 MEGA16-A, IC3 74HCT595D

Commit message: resistors moved so they wouldn't touch the SD card connector
git-svn-id: https://subversion.assembla.com/svn/atarijookie/trunk@944 0d2ca917-fb58-4453-bb26-a698c01b0940
Parts:
- moved R5 0.60 mm to (48.3, 9.50), flipped to the bottom, turned to 0 degrees
- moved R4 0.50 mm to (48.3, 11.1), flipped to the bottom, turned to 180 degrees
Routing:
- net VCC: track 166.0 -> 165.3 mm
- net N$2: track 3.20 -> 2.60 mm, vias 0 -> 1
- net LED_ACT+: track 8.61 -> 8.36 mm, vias 1 -> 0
Changed lines of the file:
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@@
 <element name="LED_PWR" library="led" package="CHIP-LED0805" value="" x="50" y="65" rot="R180"/>
 <element name="JP3" library="jumper" package="JP4" value="" x="52.5" y="10" rot="R90"/>
-<element name="R4" library="rcl" package="R0603" value="470 R" x="48.3" y="11.6"/>
+<element name="R4" library="rcl" package="R0603" value="470 R" x="48.3" y="11.1" rot="MR180"/>
 <element name="SV2" library="con-lstb" package="MA07-1" value="" x="43.4" y="17.8" rot="R180">
 <attribute name="OC_NEWARK" value="unknown" x="43.4" y="17.8" size="1.778" layer="27" rot="R180" display="off"/>
@@
 </element>
 <element name="LED_ACT" library="led" package="CHIP-LED0805" value="" x="49.4" y="6.1" rot="R180"/>
-<element name="R5" library="rcl" package="R0603" value="470 R" x="48.3" y="10.1" rot="R180"/>
+<element name="R5" library="rcl" package="R0603" value="470 R" x="48.3" y="9.5" rot="MR0"/>
 <element name="U$2" library="sd_tos" package="DIP32" value="AS6C1008DIP32" x="44.5" y="40.6"/>
 <element name="DBG" library="testpad" package="B1,27" value="TPB1,27" x="51.6" y="21.1">
@@
 <wire x1="45.9" y1="6.6" x2="45.9" y2="11" width="0.4064" layer="16"/>
 <via x="45.9" y="11" extent="1-16" drill="0.5" diameter="0.8"/>
-<wire x1="45.9" y1="11" x2="47.4" y2="11" width="0.4064" layer="1"/>
-<wire x1="47.4" y1="11" x2="47.45" y2="10.1" width="0.4064" layer="1"/>
-<wire x1="47.4" y1="10.2" x2="47.45" y2="10.1" width="0.4064" layer="1"/>
 <wire x1="38.7" y1="29.7" x2="41.7" y2="29.7" width="0.4064" layer="1"/>
 <wire x1="41.7" y1="29.7" x2="43.7" y2="29.7" width="0.4064" layer="1"/>
@@
 <wire x1="52" y1="63.9" x2="51.582003125" y2="63.9" width="0.25" layer="1"/>
 <wire x1="51.582003125" y1="63.9" x2="51.582003125" y2="60.92" width="0.4064" layer="1"/>
-<wire x1="47.45" y1="11.6" x2="47.4" y2="11.6" width="0.4064" layer="1"/>
-<wire x1="47.4" y1="11.6" x2="47.4" y2="11" width="0.4064" layer="1"/>
 <contactref element="U$1" pad="P$28"/>
-<wire x1="47.4" y1="10.2" x2="47.4" y2="11" width="0.4064" layer="1"/>
 <wire x1="52.12" y1="55.81" x2="52.12" y2="55.84" width="0.4064" layer="16"/>
 <wire x1="52.12" y1="55.84" x2="47.6" y2="55.84" width="0.4064" layer="1"/>
+<wire x1="47.45" y1="11.1" x2="47.45" y2="9.5" width="0.4064" layer="16"/>
+<wire x1="47.45" y1="11.1" x2="45.9" y2="11.1" width="0.4064" layer="16"/>
+<wire x1="45.9" y1="11.1" x2="45.9" y2="11" width="0.4064" layer="16"/>
 </signal>
 <signal name="GND">
@@
 <wire x1="50.7" y1="14.8" x2="49.2" y2="14.8" width="0.4064" layer="1"/>
 <via x="49.2" y="14.8" extent="1-16" drill="0.5" diameter="0.8"/>
-<wire x1="49.2" y1="14.8" x2="49.2" y2="12.1" width="0.4064" layer="16"/>
-<wire x1="49.2" y1="12.1" x2="52.5" y2="12.1" width="0.4064" layer="16"/>
-<wire x1="52.5" y1="12.1" x2="52.5" y2="11.27" width="0.4064" layer="16"/>
+<wire x1="49.2" y1="14.8" x2="49.2" y2="12.5" width="0.4064" layer="16"/>
+<wire x1="49.2" y1="12.5" x2="52.5" y2="12.5" width="0.4064" layer="16"/>
+<wire x1="52.5" y1="12.5" x2="52.5" y2="11.27" width="0.4064" layer="16"/>
 <wire x1="48.5" y1="25.6" x2="48.5" y2="25" width="0.4064" layer="1"/>
 <wire x1="48.5" y1="25" x2="49.4" y2="25" width="0.4064" layer="1"/>
@@
 <contactref element="R4" pad="2"/>
 <wire x1="52.5" y1="6.19" x2="52.2" y2="6.1" width="0.25" layer="16"/>
-<wire x1="52.2" y1="6.1" x2="50.4" y2="6.1" width="0.4064" layer="16"/>
-<wire x1="50.4" y1="6.1" x2="50.4" y2="11" width="0.4064" layer="16"/>
-<via x="50.4" y="11" extent="1-16" drill="0.5" diameter="0.8"/>
-<wire x1="50.4" y1="11" x2="50.05" y2="11.6" width="0.4064" layer="1"/>
-<wire x1="50.05" y1="11.6" x2="49.15" y2="11.6" width="0.4064" layer="1"/>
+<wire x1="52.2" y1="6.1" x2="50.5" y2="6.1" width="0.4064" layer="16"/>
+<wire x1="50.5" y1="6.1" x2="50.5" y2="11.1" width="0.4064" layer="16"/>
+<wire x1="50.5" y1="11.1" x2="49.15" y2="11.1" width="0.4064" layer="16"/>
 </signal>
 <signal name="N$2">
 <contactref element="R5" pad="1"/>
 <contactref element="LED_ACT" pad="A"/>
-<wire x1="49.15" y1="10.1" x2="49.15" y2="10" width="0.4064" layer="1"/>
-<wire x1="49.15" y1="10" x2="49.4" y2="10" width="0.4064" layer="1"/>
-<wire x1="49.4" y1="10" x2="49.4" y2="7.15" width="0.4064" layer="1"/>
+<wire x1="49.4" y1="7.15" x2="49.4" y2="8.2" width="0.4064" layer="1"/>
+<via x="49.4" y="8.2" extent="1-16" drill="0.5" diameter="0.8"/>
+<wire x1="49.4" y1="8.2" x2="49.4" y2="9.5" width="0.4064" layer="16"/>
+<wire x1="49.4" y1="9.5" x2="49.15" y2="9.5" width="0.4064" layer="16"/>
 </signal>
 </signals>
