File: sd_tos_hw/sd_tos_dip32.brd (EAGLE design)
At the start: 19.5 x 63.5 mm, 20 parts, among them IC1 MEGA16-A, IC3 74HCT595D

Commit message: resistors moved so they wouldn't touch the SD card connector
git-svn-id: https://subversion.assembla.com/svn/atarijookie/trunk@944 0d2ca917-fb58-4453-bb26-a698c01b0940
Parts:
- moved R5 0.30 mm to (48.4, 9.60), flipped to the bottom, turned to 0 degrees
- moved R4 0.20 mm to (48.4, 11.4), flipped to the bottom, turned to 180 degrees
Routing:
- net VCC: track 170.5 -> 169.8 mm
- net LED_ACT+: track 8.76 -> 8.96 mm, vias 1 -> 0
- net N$2: vias 0 -> 1
Changed lines of the file:
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@@
 <setting verticaltext="up"/>
 </settings>
-<grid distance="0.1" unitdist="mm" unit="mm" style="lines" multiple="1" display="yes" altdistance="0.01" altunitdist="mm" altunit="mm"/>
+<grid distance="0.1" unitdist="mm" unit="mm" style="dots" multiple="1" display="yes" altdistance="0.01" altunitdist="mm" altunit="mm"/>
 <layers>
 <layer number="1" name="Top" color="4" fill="1" visible="yes" active="yes"/>
@@
 <element name="LED_PWR" library="led" package="CHIP-LED0805" value="" x="50" y="65" rot="R180"/>
 <element name="JP3" library="jumper" package="JP4" value="" x="52.5" y="10" rot="R90"/>
-<element name="R4" library="rcl" package="R0603" value="470 R" x="48.4" y="11.6"/>
+<element name="R4" library="rcl" package="R0603" value="470 R" x="48.4" y="11.4" rot="MR180"/>
 <element name="SV2" library="con-lstb" package="MA07-1" value="" x="43.4" y="17.8" rot="R180">
 <attribute name="OC_NEWARK" value="unknown" x="43.4" y="17.8" size="1.778" layer="27" rot="R180" display="off"/>
@@
 </element>
 <element name="LED_ACT" library="led" package="CHIP-LED0805" value="" x="49.3" y="6.1" rot="R180"/>
-<element name="R5" library="rcl" package="R0603" value="470 R" x="48.4" y="9.9" rot="R180"/>
+<element name="R5" library="rcl" package="R0603" value="470 R" x="48.4" y="9.6" rot="MR0"/>
 <element name="U$2" library="sd_tos" package="DIP32" value="AS6C1008DIP32" x="44.5" y="40.6"/>
 <element name="DBG" library="testpad" package="B1,27" value="TPB1,27" x="51.6" y="21.1">
@@
 <via x="41.6" y="6.6" extent="1-16" drill="0.5" diameter="0.8"/>
 <wire x1="41.6" y1="6.6" x2="44.8" y2="6.6" width="0.4064" layer="16"/>
-<wire x1="44.8" y1="6.6" x2="44.8" y2="10.1" width="0.4064" layer="16"/>
+<wire x1="44.8" y1="6.6" x2="44.8" y2="9.5" width="0.4064" layer="16"/>
 <via x="44.8" y="10.1" extent="1-16" drill="0.5" diameter="0.8"/>
-<wire x1="44.8" y1="10.1" x2="46.6" y2="10.1" width="0.4064" layer="1"/>
-<wire x1="46.6" y1="10.1" x2="47.1" y2="10.1" width="0.4064" layer="1"/>
-<wire x1="47.1" y1="10.1" x2="47.55" y2="9.9" width="0.25" layer="1"/>
+<wire x1="44.8" y1="9.6" x2="44.8" y2="10.1" width="0.4064" layer="16"/>
 <wire x1="38.7" y1="29.7" x2="41.7" y2="29.7" width="0.4064" layer="1"/>
 <wire x1="41.7" y1="29.7" x2="43.7" y2="29.7" width="0.4064" layer="1"/>
@@
 <wire x1="52" y1="63.9" x2="51.582003125" y2="63.9" width="0.25" layer="1"/>
 <wire x1="51.582003125" y1="63.9" x2="51.582003125" y2="60.92" width="0.4064" layer="1"/>
-<wire x1="47.55" y1="11.6" x2="46.6" y2="11.6" width="0.4064" layer="1"/>
-<wire x1="46.6" y1="11.6" x2="46.6" y2="10.1" width="0.4064" layer="1"/>
+<wire x1="47.55" y1="11.4" x2="47.55" y2="9.6" width="0.4064" layer="16"/>
+<wire x1="47.55" y1="9.6" x2="44.8" y2="9.6" width="0.4064" layer="16"/>
+<wire x1="44.8" y1="9.6" x2="44.8" y2="9.5" width="0.4064" layer="16"/>
 </signal>
 <signal name="GND">
@@
 <contactref element="R4" pad="2"/>
 <wire x1="52.5" y1="6.19" x2="52.2" y2="6.1" width="0.25" layer="16"/>
-<wire x1="52.2" y1="6.1" x2="50.3" y2="6.1" width="0.4064" layer="16"/>
-<wire x1="50.3" y1="6.1" x2="50.3" y2="11.3" width="0.4064" layer="16"/>
-<via x="50.3" y="11.3" extent="1-16" drill="0.5" diameter="0.8"/>
-<wire x1="50.3" y1="11.3" x2="50.3" y2="11.6" width="0.4064" layer="1"/>
-<wire x1="50.3" y1="11.6" x2="49.25" y2="11.6" width="0.4064" layer="1"/>
+<wire x1="52.2" y1="6.1" x2="50.5" y2="6.1" width="0.4064" layer="16"/>
+<wire x1="50.5" y1="11.6" x2="49.25" y2="11.6" width="0.4064" layer="16"/>
+<wire x1="49.25" y1="11.6" x2="49.25" y2="11.4" width="0.4064" layer="16"/>
+<wire x1="50.5" y1="6.1" x2="50.5" y2="11.6" width="0.4064" layer="16"/>
 </signal>
 <signal name="N$2">
 <contactref element="R5" pad="1"/>
 <contactref element="LED_ACT" pad="A"/>
-<wire x1="49.25" y1="9.9" x2="49.3" y2="9.9" width="0.4064" layer="1"/>
-<wire x1="49.3" y1="9.9" x2="49.3" y2="7.15" width="0.4064" layer="1"/>
+<wire x1="49.25" y1="9.6" x2="49.3" y2="9.9" width="0.4064" layer="16"/>
+<wire x1="49.3" y1="7.15" x2="49.3" y2="8.5" width="0.4064" layer="1"/>
+<via x="49.3" y="8.5" extent="1-16" drill="0.5" diameter="0.8"/>
+<wire x1="49.3" y1="8.5" x2="49.25" y2="8.5" width="0.4064" layer="16"/>
+<wire x1="49.25" y1="8.5" x2="49.25" y2="9.6" width="0.4064" layer="16"/>
 </signal>
 </signals>
